File: zx-sdc-v0.1.kicad_sch (KiCad schematic)
At the start: 65 parts, among them J1 SD_Card, J2 Micro_SD_Card_Det2, J3 Conn_01x02_Pin, Q1 2N7000, Q2 BC557, U1 74LS688, U10 74LS125, U11 74LS595, U12 74LS30, U13 74LS138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

Commit message: - added time diagram  - created backup v0.1  - created backup v0.2  - added various changes
Parts:
- removed U12: 74LS30, symbol 74xx:74LS30
- removed U13: 74LS138, symbol 74xx:74LS138
- C3: value 10u -> 220u
- C4: value 4u7 -> 220u
Connections:
- net +5V: now also U1.14 (R5)
- net A3: no longer U6.11
- net A7: no longer U6.13
- net /M1: no longer names the net of Z1.A24 (~{M1})
- net /M1: no longer U1.14 (R5)
- no-connect marks 52 -> 23
Other:
- note removed: "0x77 control port Bit 0: sd power 0=off,1=on Bit 1: sd cs 0=selected,1=deselected Bit 2-7: unused 0x57 data port - SPI rd/wr"
- moved on the sheet: D1, D2, D3, Q2, R1, R15, R2, R22, R3, R5, U10C, U8A
