File: zx-sdc-v0.2.kicad_sch (KiCad schematic)
At the start: 65 parts, among them J1 SD_Card, J2 Micro_SD_Card_Det2, J3 Conn_01x02_Pin, Q1 2N7000, Q2 BC557, U1 74LS688, U10 74LS125, U11 74LS595, U12 74LS30, U13 74LS138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

Commit message: - added time diagram  - created backup v0.1  - created backup v0.2  - added various changes
Parts:
- removed U12: 74LS30, symbol 74xx:74LS30
- removed U13: 74LS138, symbol 74xx:74LS138
- removed U6: 74LS04, symbol 74xx:74LS04
- added U12: 74LS00, symbol 74xx:74LS00
Connections:
- net +5V: now also U12.14 (VCC)
- net AUX_CLK: now also U12.6
- net DONE: now also U12.12, U12.13
- net GND: now also U12.7 (GND)
- net SPI_CLK: now also U12.10, U12.9
- net /DONE: now also U12.11
- net /SPI_CLK: now also U12.8
- net at R1.2, R2.1: now also U12.3, U12.4, U12.5
- net at R1.1, Y1.1: now also U12.1, U12.2
- no-connect marks 52 -> 48
Other:
- note removed: "0x77 control port Bit 0: sd power 0=off,1=on Bit 1: sd cs 0=selected,1=deselected Bit 2-7: unused 0x57 data port - SPI rd/wr"
