File: zx-sdc.kicad_pcb (KiCad board)
At the start: 2 copper layers, 80 x 125.7 mm, 67 parts, among them J1 SD_Card, J2 Micro_SD_Card_Det2, J4 Conn_01x03_Pin, Q1 2N7000, Q2 BC557, U10 74LS125, U11 74LS595, U12 74LS30, U13 74LS138, U3 AMS1117-3.3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

Commit message: refinings & last cuts
Other:
- board text added: "${COMMENT1}"
- board text added: "${COMMENT2} ${ISSUE_DATE}"
- board text added: "${TITLE} Rev: ${REVISION}"
- board text added: "Designed by ${COMPANY}"
- board text removed: "Designed by Maksym / 7FFD"
- board text removed: "KYIV, UKRAINE 01.10.2024"
- board text removed: "ZX SDC / Hardware version of z-controller"
- board text removed: "http://7ffd.geektimes.eu/"
Changed lines of the file:
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@@
   )
   (paper "A4")
+  (title_block
+    (title "ZX SDC / Hardware version of z-controller")
+    (date "2024-10-01")
+    (rev "0.1")
+    (company "Maksym / 7FFD")
+    (comment 1 "http://7ffd.geektimes.eu/")
+    (comment 2 "KYIV, UKRAINE")
+  )
   (layers
     (0 "F.Cu" signal)
@@
   (gr_line (start 63.4365 165.1635) (end 65.9765 165.1635)
     (stroke (width 0.1) (type default)) (layer "Edge.Cuts"))
-  (gr_text "http://7ffd.geektimes.eu/" (at 112.522 41.402) (layer "F.SilkS")
+  (gr_text "${COMMENT1}" (at 112.522 41.402) (layer "F.SilkS")
     (effects (font (size 1.5 1.5) (thickness 0.15)) (justify left bottom))
   )
-  (gr_text "KYIV, UKRAINE 01.10.2024" (at 142.748 82.042 90) (layer "F.SilkS")
+  (gr_text "${COMMENT2} ${ISSUE_DATE}" (at 142.875 75.819 90) (layer "F.SilkS")
     (effects (font (size 1.5 1.5) (thickness 0.15)) (justify left bottom))
   )
-  (gr_text "Designed by Maksym / 7FFD" (at 66.421 140.081 90) (layer "F.SilkS")
+  (gr_text "Designed by ${COMPANY}" (at 66.421 140.081 90) (layer "F.SilkS")
     (effects (font (size 2 2) (thickness 0.15)) (justify left bottom))
   )
-  (gr_text "ZX SDC / Hardware version of z-controller" (at 142.748 139.573 90) (layer "F.SilkS")
+  (gr_text "${TITLE} Rev: ${REVISION}" (at 142.748 139.573 90) (layer "F.SilkS")
     (effects (font (size 1.5 1.5) (thickness 0.15)) (justify left bottom))
   )
